File: computerScienceExperience2/computerScienceExperience2.kicad_pcb (KiCad board)
At the start: 2 copper layers, 121 parts, among them J1 Conn_01x02, SW1 SW_Push_SPDT, SW2 SW_DIP_x02, U1 74HC73, U2 74HC04, U3 74HC00

Commit message: computerScienceExperience2 ver1.10
Parts:
- removed the G*** at (109.1, 71.4)
Other:
- board outline added: 98.9 x 96.1 mm
- board text added: "2019/11/12 ver. 1.10"
- board text added: "V-CUT"
- board text removed: "2019/11/07 ver. 1.00"

Commit message: computerScienceExperience2 ver1.20
Parts:
- removed the SW1 at (124.0, 75.5)
- added D1: LED, LED_SMD:LED_0603_1608Metric_Pad1.05x0.95mm_HandSolder, F.Cu at (84.8, 29.1)
- added D2: LED, LED_SMD:LED_0603_1608Metric_Pad1.05x0.95mm_HandSolder, F.Cu at (87.3, 29.1)
- added D3: LED, LED_SMD:LED_0603_1608Metric_Pad1.05x0.95mm_HandSolder, F.Cu at (90.6, 24.6)
- added G***: LOGO, Downloads:cit_logo, F.Cu at (52.3, 34.9)
- added J1: Conn_01x02, Connector_PinHeader_2.54mm:PinHeader_1x02_P2.54mm_Vertical, F.Cu at (46.6, 25.7)
- added R1: 470, Resistor_SMD:R_0603_1608Metric_Pad1.05x0.95mm_HandSolder, F.Cu at (51.6, 23.2)
- added R2: 470, Resistor_SMD:R_0603_1608Metric_Pad1.05x0.95mm_HandSolder, F.Cu at (51.6, 26.2)
- added R3: 470, Resistor_SMD:R_0603_1608Metric_Pad1.05x0.95mm_HandSolder, F.Cu at (84.8, 24.6)
- added R4: 470, Resistor_SMD:R_0603_1608Metric_Pad1.05x0.95mm_HandSolder, F.Cu at (87.3, 24.6)
- added R5: 470, Resistor_SMD:R_0603_1608Metric_Pad1.05x0.95mm_HandSolder, F.Cu at (90.6, 29.1)
- added SW1: SW_Push_SPDT-ALT, myFootprints:TL2285, F.Cu at (124.0, 75.5)
- added SW1: SW_Push_SPDT-ALT, myFootprints:TL2285, F.Cu at (66.1, 38.2)
- added SW2: SW_DIP_x02, Package_DIP:DIP-4_W7.62mm_SMDSocket_SmallPads, F.Cu at (79.1, 38.5)
- added U1: 74HC73, myFootprints:74HC73D_14-SOIC, F.Cu at (69.8, 27.0)
- added U2: 74HC04, myFootprints:74HC04D_14-SOIC, F.Cu at (79.6, 27.0)
- added U3: 74HC00, myFootprints:74HC00D_14-SOIC, F.Cu at (59.8, 27.0)
- SW1 (x7): value SW_Push_SPDT -> SW_Push_SPDT-ALT
Connections:
- SW1 pad 2: /GND -> Net-(R2-Pad2) (x7)
- SW1 pad 3: Net-(R2-Pad2) -> /GND (x7)
Routing:
- net /GND: track 493.4 -> 567.1 mm, vias 32 -> 36
- net /Vcc: track 586.0 -> 659.2 mm
- net /INPUT_K: track 282.7 -> 318.1 mm, vias 16 -> 18
- net /INPUT_J: track 243.7 -> 274.3 mm, vias 16 -> 18
- net Net-(R5-Pad2): track 201.5 -> 226.7 mm, vias 16 -> 18
- net Net-(R1-Pad2): track 201.0 -> 226.1 mm, vias 16 -> 18
- net Net-(R2-Pad2): track 210.4 -> 234.4 mm, vias 16 -> 18
- net /CLK: track 190.1 -> 213.9 mm
- net /OUTPUT_Q: track 86.9 -> 97.8 mm
- net Net-(U3-Pad3): track 35.1 -> 39.5 mm
- net Net-(D3-Pad1): track 22.0 -> 24.8 mm
- net Net-(D2-Pad2): track 22.0 -> 24.8 mm
- net Net-(D1-Pad2): track 22.0 -> 24.8 mm
Other:
- board size 98.9 x 96.1 mm -> 156.5 x 133.4 mm
- board text added: "2019/11/27 ver. 1.20"

Commit message: computerScienceExperence2 ver. 2.00
Parts:
- removed the D1 at (142.8, 66.4)
- removed the D1 at (142.8, 138.4)
- removed the D1 at (192.2, 138.4)
- removed the D1 at (142.8, 90.4)
- removed the D1 at (192.2, 114.4)
- removed the D1 at (192.2, 66.4)
- removed the D1 at (142.8, 114.4)
- removed the D1 at (192.2, 90.4)
- removed the D1 at (84.8, 29.1)
- removed the D2 at (145.2, 66.4)
- removed the D2 at (145.2, 138.4)
- removed the D2 at (194.8, 66.4)
- removed the D2 at (194.8, 114.4)
- removed the D2 at (194.8, 90.4)
- removed the D2 at (145.2, 90.4)
- removed the D2 at (145.2, 114.4)
- removed the D2 at (194.8, 138.4)
- removed the D2 at (87.3, 29.1)
- removed the D3 at (148.5, 61.9)
- removed the D3 at (198.0, 85.9)
- removed the D3 at (148.5, 85.9)
- removed the D3 at (148.5, 109.9)
- removed the D3 at (198.0, 61.9)
- removed the D3 at (198.0, 109.9)
- removed the D3 at (148.5, 133.9)
- removed the D3 at (198.0, 133.9)
- removed the D3 at (90.6, 24.6)
- removed the G*** at (110.2, 144.2)
- removed the G*** at (159.7, 144.2)
- removed the G*** at (159.7, 72.2)
- removed the G*** at (110.2, 120.2)
- removed the G*** at (110.2, 72.2)
- removed the G*** at (159.7, 96.2)
- removed the G*** at (110.2, 96.2)
- removed the G*** at (159.7, 120.2)
- removed the G*** at (52.3, 34.9)
- removed the J1 at (104.5, 111.0)
- removed the J1 at (104.5, 87.0)
- removed the J1 at (154.0, 63.0)
- removed the J1 at (104.5, 135.0)
- removed the J1 at (154.0, 111.0)
- removed the J1 at (154.0, 87.0)
- removed the J1 at (104.5, 63.0)
- removed the J1 at (154.0, 135.0)
- removed the J1 at (46.6, 25.7)
- removed the R1 at (109.5, 60.5)
- removed the R1 at (159.0, 132.5)
- removed the R1 at (109.5, 108.5)
- removed the R1 at (109.5, 84.5)
- removed the R1 at (159.0, 60.5)
- removed the R1 at (159.0, 84.5)
- removed the R1 at (109.5, 132.5)
- removed the R1 at (159.0, 108.5)
- removed the R1 at (51.6, 23.2)
- removed the R2 at (109.5, 111.5)
- removed the R2 at (109.5, 63.5)
- removed the R2 at (159.0, 135.5)
- removed the R2 at (109.5, 135.5)
- removed the R2 at (159.0, 87.5)
- removed the R2 at (109.5, 87.5)
- removed the R2 at (159.0, 63.5)
- removed the R2 at (159.0, 111.5)
- removed the R2 at (51.6, 26.2)
- removed the R3 at (142.8, 85.9)
- removed the R3 at (142.8, 61.9)
- removed the R3 at (142.8, 133.9)
- removed the R3 at (192.2, 85.9)
- removed the R3 at (192.2, 133.9)
- removed the R3 at (142.8, 109.9)
- removed the R3 at (192.2, 61.9)
- removed the R3 at (192.2, 109.9)
- removed the R3 at (84.8, 24.6)
- removed the R4 at (194.8, 109.9)
- removed the R4 at (145.2, 61.9)
- removed the R4 at (145.2, 133.9)
- removed the R4 at (194.8, 61.9)
- removed the R4 at (145.2, 109.9)
- removed the R4 at (194.8, 133.9)
- removed the R4 at (145.2, 85.9)
- removed the R4 at (194.8, 85.9)
- removed the R4 at (87.3, 24.6)
- removed the R5 at (148.5, 138.4)
- removed the R5 at (148.5, 66.4)
- removed the R5 at (198.0, 114.4)
- removed the R5 at (148.5, 90.4)
- removed the R5 at (198.0, 90.4)
- removed the R5 at (198.0, 66.4)
- removed the R5 at (198.0, 138.4)
- removed the R5 at (148.5, 114.4)
- removed the R5 at (90.6, 29.1)
- removed the SW1 at (124.0, 147.5)
- removed the SW1 at (173.5, 75.5)
- removed the SW1 at (124.0, 99.5)
- removed the SW1 at (173.5, 123.5)
- removed the SW1 at (124.0, 123.5)
- removed the SW1 at (173.5, 99.5)
- removed the SW1 at (173.5, 147.5)
- removed the SW1 at (124.0, 75.5)
- removed the SW1 at (66.1, 38.2)
- removed the SW2 at (137.0, 147.8)
- removed the SW2 at (186.5, 123.8)
- removed the SW2 at (137.0, 99.8)
- removed the SW2 at (137.0, 123.8)
- removed the SW2 at (137.0, 75.8)
- removed the SW2 at (186.5, 147.8)
- removed the SW2 at (186.5, 75.8)
- removed the SW2 at (186.5, 99.8)
- removed the SW2 at (79.1, 38.5)
- removed U1 (x9): 74HC73, myFootprints:74HC73D_14-SOIC
- removed U2 (x9): 74HC04, myFootprints:74HC04D_14-SOIC
- removed U3 (x9): 74HC00, myFootprints:74HC00D_14-SOIC
- added 74LS00: 74HC00, Package_DIP:DIP-14_W8.89mm_SMDSocket_LongPads, F.Cu at (117.9, 64.6)
- added 74LS04: 74HC04, Package_DIP:DIP-14_W8.89mm_SMDSocket_LongPads, F.Cu at (147.6, 64.6)
- added 74LS73: 74HC73, Package_DIP:DIP-14_W8.89mm_SMDSocket_LongPads, F.Cu at (132.7, 64.6)
- added CLK: Conn_01x01_Male, Connector_PinHeader_2.54mm:PinHeader_1x01_P2.54mm_Vertical, F.Cu at (128.3, 53.4)
- added D1: LED, LED_SMD:LED_1206_3216Metric_Pad1.42x1.75mm_HandSolder, F.Cu at (157.9, 62.2)
- added D2: LED, LED_SMD:LED_1206_3216Metric_Pad1.42x1.75mm_HandSolder, F.Cu at (161.8, 62.2)
- added D3: LED, LED_SMD:LED_1206_3216Metric_Pad1.42x1.75mm_HandSolder, F.Cu at (167.2, 55.0)
- added G***: LOGO, myFootprints:cit_logo, F.Cu at (100.2, 71.7)
- added J1: Conn_01x02, Connector_PinHeader_2.54mm:PinHeader_1x02_P2.54mm_Vertical, F.Cu at (99.5, 55.6)
- added Q: Conn_01x01_Male, Connector_PinHeader_2.54mm:PinHeader_1x01_P2.54mm_Vertical, F.Cu at (137.2, 53.4)
- added R1: 470, Resistor_SMD:R_1206_3216Metric_Pad1.42x1.75mm_HandSolder, F.Cu at (106.3, 53.1)
- added R2: 470, Resistor_SMD:R_1206_3216Metric_Pad1.42x1.75mm_HandSolder, F.Cu at (106.3, 56.7)
- added R3: 470, Resistor_SMD:R_1206_3216Metric_Pad1.42x1.75mm_HandSolder, F.Cu at (157.9, 55.0)
- added R4: 470, Resistor_SMD:R_1206_3216Metric_Pad1.42x1.75mm_HandSolder, F.Cu at (161.8, 55.0)
- added R5: 470, Resistor_SMD:R_1206_3216Metric_Pad1.42x1.75mm_HandSolder, F.Cu at (167.2, 62.2)
- added SW1: SW_Push_SPDT, myFootprints:TL2285, F.Cu at (103.3, 63.7)
- added SW2: SW_DIP_x02, Package_DIP:DIP-4_W8.89mm_SMDSocket_LongPads, F.Cu at (162.1, 70.3)
Routing:
- net /Vcc: track 659.2 -> 33.0 mm
- net /GND: track 567.1 -> 116.3 mm, vias 36 -> 2
- net /INPUT_K: track 318.1 -> 50.5 mm, vias 18 -> 4
- net Net-(R2-Pad2): track 234.4 -> 16.1 mm, vias 18 -> 2
- net /INPUT_J: track 274.3 -> 57.6 mm, vias 18 -> 3
- net Net-(R1-Pad2): track 226.1 -> 20.4 mm, vias 18 -> 2
- net Net-(R5-Pad2): track 226.7 -> 37.5 mm, vias 18 -> 2
- net /CLK: track 213.9 -> 36.2 mm, vias 0 -> 2
- net /OUTPUT_Q: track 97.8 -> 24.4 mm, vias 0 -> 2
- net Net-(U3-Pad3): track 39.5 -> 7.18 mm
- net Net-(D3-Pad1): track 24.8 -> 4.22 mm
- net Net-(D1-Pad2): track 24.8 -> 4.23 mm
- net Net-(D2-Pad2): track 24.8 -> 4.23 mm
- net /OUTPUT_PULSE: track 0.00 -> 15.6 mm
- net /PULSE: track 0.00 -> 3.62 mm
Other:
- board outline removed
- board text added: "20191130 Ver. 2.00"
- board text added: "INPUT"
- board text added: "OUTPUT"
- board text removed: "2019/11/12 ver. 1.10"
- board text removed: "2019/11/27 ver. 1.20"
- board text removed: "74HC00"
- board text removed: "74HC04"
- board text removed: "74HC73"
- board text removed: "IN"
- board text removed: "J"
- board text removed: "K"
- board text removed: "KiCad 5.1.4 FusionPCB"
- board text removed: "OUT"
- board text removed: "V-CUT"
