File: computerScienceExperience2/computerScienceExperience2.sch (KiCad schematic (older format))
At the start: 14 parts, among them J1 Conn_01x02, SW1 SW_Push_SPDT, SW2 SW_DIP_x02, U1 74HC73, U2 74HC04, U3 74HC00

Commit message: computerScienceExperience2 ver1.20
Parts:
- removed SW1: SW_Push_SPDT, myFootprints:TL2285, symbol Switch:SW_Push_SPDT
- added SW1: SW_Push_SPDT-ALT, myFootprints:TL2285, symbol myComponents:SW_Push_SPDT-ALT
Connections:
- net GND: now also SW1.3 (C)
- net at R1.2, U3.1: now also SW1.1 (A)
- net at R2.2, U3.5: now also SW1.2 (B)
Other:
- moved on the sheet: U1B, U1C, U3E
Changed lines of the file:
@@
 Wire Wire Line
 	6600 3500 5950 3500
-$Comp
-L Switch:SW_Push_SPDT SW1
-U 1 1 5DC7392C
-P 6050 4550
-F 0 "SW1" V 6096 4362 50  0000 R CNN
-F 1 "SW_Push_SPDT" V 6005 4362 50  0000 R CNN
-F 2 "myFootprints:TL2285" H 6050 4550 50  0001 C CNN
-F 3 "~" H 6050 4550 50  0001 C CNN
-	1    6050 4550
-	0    -1   -1   0
-$EndComp
 Wire Wire Line
 	6150 4200 6150 4350
@@
 Wire Bus Line
 	5600 2700 5600 5000
-Wire Bus Line
-	5600 5000 7900 5000
-Wire Bus Line
-	7900 5000 7900 2700
-Wire Bus Line
-	7900 2700 5600 2700
 Text Notes 6400 5150 0    50   ~ 0
 Pulse Generater
-Text Label 9200 3550 0    50   ~ 0
-OUTPUT_Q
-Text Label 8600 3750 2    50   ~ 0
-INPUT_K
-Text Label 8600 3650 2    50   ~ 0
-CLK
-Text Label 8600 3550 2    50   ~ 0
-INPUT_J
-NoConn ~ 9200 3750
-Wire Bus Line
-	8250 3400 8250 4550
-Wire Bus Line
-	8250 4550 9600 4550
-Wire Bus Line
-	9600 4550 9600 3400
-Wire Bus Line
-	9600 3400 8250 3400
-Text Notes 8700 4650 0    50   ~ 0
-JK FlipFlop
 $Comp
 L Device:R R4
@@
 Text Label 6050 4900 0    50   ~ 0
 GND
-Text Label 8900 3950 0    50   ~ 0
-Vcc
 $Comp
 L power:PWR_FLAG #FLG0102
@@
 Text Notes 2550 3400 0    50   ~ 0
 Power
-$Comp
-L myComponents:74HC73 U1
-U 3 1 5E0F5F4C
-P 8850 4350
-F 0 "U1" V 9167 4300 50  0000 C CNN
-F 1 "74HC73" V 9076 4300 50  0000 C CNN
-F 2 "myFootprints:74HC73D_14-SOIC" H 8500 4700 50  0001 C CNN
-F 3 "" H 8500 4700 50  0001 C CNN
-	3    8850 4350
-	0    -1   -1   0
-$EndComp
-Text Label 9200 4350 0    50   ~ 0
-GND
-Text Label 8600 4350 2    50   ~ 0
-Vcc
-$Comp
-L 74xx:74HC00 U3
-U 5 1 5E1277B6
-P 7200 4750
-F 0 "U3" V 7567 4750 50  0000 C CNN
-F 1 "74HC00" V 7476 4750 50  0000 C CNN
-F 2 "myFootprints:74HC00D_14-SOIC" H 7200 4750 50  0001 C CNN
-F 3 "http://www.ti.com/lit/gpn/sn74hc00" H 7200 4750 50  0001 C CNN
-	5    7200 4750
-	0    -1   -1   0
-$EndComp
 Text Label 2450 4900 2    50   ~ 0
 OUTPUT_Q
-Text Label 6700 4750 2    50   ~ 0
-Vcc
-Text Label 7700 4750 0    50   ~ 0
-GND
-$Comp
-L myComponents:74HC73 U1
-U 2 1 5E19F83D
-P 8900 3650
-F 0 "U1" H 9129 10715 50  0000 C CNN
-F 1 "74HC73" H 9129 10624 50  0000 C CNN
-F 2 "myFootprints:74HC73D_14-SOIC" H 8550 4000 50  0001 C CNN
-F 3 "" H 8550 4000 50  0001 C CNN
-	2    8900 3650
-	1    0    0    -1
-$EndComp
 $Comp
 L 74xx:74HC04 U2
@@
 Text Label 2950 4250 0    50   ~ 0
 GND
+$Comp
+L myComponents:SW_Push_SPDT-ALT SW1
+U 1 1 5DDF5F97
+P 6050 4550
+F 0 "SW1" V 6096 4362 50  0000 R CNN
+F 1 "SW_Push_SPDT-ALT" V 6005 4362 50  0000 R CNN
+F 2 "myFootprints:TL2285" H 6050 4550 50  0001 C CNN
+F 3 "~" H 6050 4550 50  0001 C CNN
+	1    6050 4550
+	0    -1   -1   0
+$EndComp
+Wire Bus Line
+	8100 5000 8100 2700
+Wire Bus Line
+	5600 5000 8100 5000
+Wire Bus Line
+	8100 2700 5600 2700
+$Comp
+L 74xx:74HC00 U3
+U 5 1 5E1277B6
+P 7350 4750
+F 0 "U3" V 7717 4750 50  0000 C CNN
+F 1 "74HC00" V 7626 4750 50  0000 C CNN
+F 2 "myFootprints:74HC00D_14-SOIC" H 7350 4750 50  0001 C CNN
+F 3 "http://www.ti.com/lit/gpn/sn74hc00" H 7350 4750 50  0001 C CNN
+	5    7350 4750
+	0    -1   -1   0
+$EndComp
+Text Label 6850 4750 2    50   ~ 0
+Vcc
+Text Label 7850 4750 0    50   ~ 0
+GND
+Text Label 9350 3550 0    50   ~ 0
+OUTPUT_Q
+Text Label 8750 3750 2    50   ~ 0
+INPUT_K
+Text Label 8750 3650 2    50   ~ 0
+CLK
+Text Label 8750 3550 2    50   ~ 0
+INPUT_J
+NoConn ~ 9350 3750
+Wire Bus Line
+	8400 3400 8400 4550
+Wire Bus Line
+	8400 4550 9750 4550
+Wire Bus Line
+	9750 4550 9750 3400
+Wire Bus Line
+	9750 3400 8400 3400
+Text Notes 8850 4650 0    50   ~ 0
+JK FlipFlop
+Text Label 9050 3950 0    50   ~ 0
+Vcc
+$Comp
+L myComponents:74HC73 U1
+U 3 1 5E0F5F4C
+P 9000 4350
+F 0 "U1" V 9317 4300 50  0000 C CNN
+F 1 "74HC73" V 9226 4300 50  0000 C CNN
+F 2 "myFootprints:74HC73D_14-SOIC" H 8650 4700 50  0001 C CNN
+F 3 "" H 8650 4700 50  0001 C CNN
+	3    9000 4350
+	0    -1   -1   0
+$EndComp
+Text Label 9350 4350 0    50   ~ 0
+GND
+Text Label 8750 4350 2    50   ~ 0
+Vcc
+$Comp
+L myComponents:74HC73 U1
+U 2 1 5E19F83D
+P 9050 3650
+F 0 "U1" H 9279 10715 50  0000 C CNN
+F 1 "74HC73" H 9279 10624 50  0000 C CNN
+F 2 "myFootprints:74HC73D_14-SOIC" H 8700 4000 50  0001 C CNN
+F 3 "" H 8700 4000 50  0001 C CNN
+	2    9050 3650
+	1    0    0    -1
+$EndComp
 $EndSCHEMATC

Commit message: computerScienceExperence2 ver. 2.00
Parts:
- removed SW1: SW_Push_SPDT-ALT, myFootprints:TL2285, symbol myComponents:SW_Push_SPDT-ALT
- added J2, J3: Conn_01x01_Male, Connector_PinHeader_2.54mm:PinHeader_1x01_P2.54mm_Vertical, symbol Connector:Conn_01x01_Male
- added SW1: SW_Push_SPDT, myFootprints:TL2285, symbol Switch:SW_Push_SPDT
- added unit 1 of U1
- D1, D2, D3: footprint LED_SMD:LED_0603_1608Metric_Pad1.05x0.95mm_HandSolder -> LED_SMD:LED_1206_3216Metric_Pad1.42x1.75mm_HandSolder
- R1, R2, R3, R4, R5: footprint Resistor_SMD:R_0603_1608Metric_Pad1.05x0.95mm_HandSolder -> Resistor_SMD:R_1206_3216Metric_Pad1.42x1.75mm_HandSolder
- SW2: footprint Package_DIP:DIP-4_W7.62mm_SMDSocket_SmallPads -> Package_DIP:DIP-4_W8.89mm_SMDSocket_LongPads
- U1: footprint myFootprints:74HC73D_14-SOIC -> Package_DIP:DIP-14_W8.89mm_SMDSocket_LongPads
- U2: footprint myFootprints:74HC04D_14-SOIC -> Package_DIP:DIP-14_W8.89mm_SMDSocket_LongPads
- U3: footprint myFootprints:74HC00D_14-SOIC -> Package_DIP:DIP-14_W8.89mm_SMDSocket_LongPads
Connections:
- net GND: now also SW1.2 (B)
- net Vcc: now also U1.14 (J), U1.2 (~R), U1.3 (K)
- net at R1.2, U3.1: now also SW1.1 (A)
- net at R2.2, U3.5: now also SW1.3 (C)
- new net OUTPUT_PULSE: J2.1 (Pin_1), U1.12 (Q)
- new net PULSE: J3.1 (Pin_1), U1.1 (~CP)
- no-connect marks 1 -> 2
Other:
- note added: "PULSE"
- moved on the sheet: D3, R1, R2, R5, U1C, U2A, U2G, U3A, U3B, U3E
