File: cse2/circuit-2/circuit-2.sch (KiCad schematic (older format))
At the start: 7 parts, among them J1 Conn_01x01_Male, J2 Conn_01x01_Male, J3 Conn_01x01_Male, J4 Conn_01x01_Male, J5 Conn_01x01_Male, U1 74LS73, U2 74LS00

Commit message: complete circuit-2
Parts:
- J1, J2, J5: footprint Connector_Pin:Pin_D1.4mm_L8.5mm_W2.8mm_FlatFork -> Connector_PinHeader_2.54mm:PinHeader_1x01_P2.54mm_Vertical
- U1, U2: footprint Connector_PinSocket_2.54mm:PinSocket_2x07_P2.54mm_Vertical -> myFootprint:DIP-14-SMD
Connections:
- net CK: now also U1.1 (C); no longer U1.5 (C)
- net at J3.1 (Pin_1), U2.1: now also U1.12 (Q), U1.5 (C); no longer U1.1 (C), U1.9 (Q)
- net at J4.1 (Pin_1), U2.2: now also U1.9 (Q); no longer U1.12 (Q)
Other:
- moved on the sheet: U1A, U1B
Changed lines of the file:
@@
 L 74xx:74LS73 U1
 U 1 1 5F60DCD7
+P 4700 1950
+F 0 "U1" V 4654 2180 50  0000 L CNN
+F 1 "74LS73" V 4745 2180 50  0000 L CNN
+F 2 "myFootprint:DIP-14-SMD" H 4700 1950 50  0001 C CNN
+F 3 "http://www.ti.com/lit/gpn/sn74LS73" H 4700 1950 50  0001 C CNN
+	1    4700 1950
+	0    1    1    0
+$EndComp
+$Comp
+L 74xx:74LS73 U1
+U 2 1 5F60E814
 P 5650 1950
 F 0 "U1" V 5604 2180 50  0000 L CNN
 F 1 "74LS73" V 5695 2180 50  0000 L CNN
-F 2 "Connector_PinSocket_2.54mm:PinSocket_2x07_P2.54mm_Vertical" H 5650 1950 50  0001 C CNN
+F 2 "myFootprint:DIP-14-SMD" H 5650 1950 50  0001 C CNN
 F 3 "http://www.ti.com/lit/gpn/sn74LS73" H 5650 1950 50  0001 C CNN
-	1    5650 1950
-	0    1    1    0
-$EndComp
-$Comp
-L 74xx:74LS73 U1
-U 2 1 5F60E814
-P 4700 1950
-F 0 "U1" V 4654 2180 50  0000 L CNN
-F 1 "74LS73" V 4745 2180 50  0000 L CNN
-F 2 "Connector_PinSocket_2.54mm:PinSocket_2x07_P2.54mm_Vertical" H 4700 1950 50  0001 C CNN
-F 3 "http://www.ti.com/lit/gpn/sn74LS73" H 4700 1950 50  0001 C CNN
-	2    4700 1950
+	2    5650 1950
 	0    1    1    0
 $EndComp
@@
 F 0 "U1" V 2517 2950 50  0000 C CNN
 F 1 "74LS73" V 2426 2950 50  0000 C CNN
-F 2 "Connector_PinSocket_2.54mm:PinSocket_2x07_P2.54mm_Vertical" H 2150 2950 50  0001 C CNN
+F 2 "myFootprint:DIP-14-SMD" H 2150 2950 50  0001 C CNN
 F 3 "http://www.ti.com/lit/gpn/sn74LS73" H 2150 2950 50  0001 C CNN
 	3    2150 2950
@@
 F 0 "J2" H 1450 5100 50  0000 L CNN
 F 1 "Conn_01x01_Male" H 1150 5000 50  0000 L CNN
-F 2 "Connector_Pin:Pin_D1.4mm_L8.5mm_W2.8mm_FlatFork" H 1400 4900 50  0001 C CNN
+F 2 "Connector_PinHeader_2.54mm:PinHeader_1x01_P2.54mm_Vertical" H 1400 4900 50  0001 C CNN
 F 3 "~" H 1400 4900 50  0001 C CNN
 	1    1400 4900
@@
 F 0 "U2" V 5604 3088 50  0000 L CNN
 F 1 "74LS00" V 5695 3088 50  0000 L CNN
-F 2 "Connector_PinSocket_2.54mm:PinSocket_2x07_P2.54mm_Vertical" H 5650 2900 50  0001 C CNN
+F 2 "myFootprint:DIP-14-SMD" H 5650 2900 50  0001 C CNN
 F 3 "http://www.ti.com/lit/gpn/sn74ls00" H 5650 2900 50  0001 C CNN
 	1    5650 2900
@@
 F 0 "U2" V 2517 3650 50  0000 C CNN
 F 1 "74LS00" V 2426 3650 50  0000 C CNN
-F 2 "Connector_PinSocket_2.54mm:PinSocket_2x07_P2.54mm_Vertical" H 2150 3650 50  0001 C CNN
+F 2 "myFootprint:DIP-14-SMD" H 2150 3650 50  0001 C CNN
 F 3 "http://www.ti.com/lit/gpn/sn74ls00" H 2150 3650 50  0001 C CNN
 	5    2150 3650
@@
 F 0 "J1" H 1408 1531 50  0000 C CNN
 F 1 "Conn_01x01_Male" H 1408 1440 50  0000 C CNN
-F 2 "Connector_Pin:Pin_D1.4mm_L8.5mm_W2.8mm_FlatFork" H 1300 1350 50  0001 C CNN
+F 2 "Connector_PinHeader_2.54mm:PinHeader_1x01_P2.54mm_Vertical" H 1300 1350 50  0001 C CNN
 F 3 "~" H 1300 1350 50  0001 C CNN
 	1    1300 1350
@@
 F 0 "J5" H 1408 1631 50  0000 C CNN
 F 1 "Conn_01x01_Male" H 1408 1540 50  0000 C CNN
-F 2 "Connector_Pin:Pin_D1.4mm_L8.5mm_W2.8mm_FlatFork" H 1300 1450 50  0001 C CNN
+F 2 "Connector_PinHeader_2.54mm:PinHeader_1x01_P2.54mm_Vertical" H 1300 1450 50  0001 C CNN
 F 3 "~" H 1300 1450 50  0001 C CNN
 	1    1300 1450
