File: cse2/circuit-2/circuit-2.kicad_pcb (KiCad board)
At the start: 2 copper layers, 8 parts, among them Q0 Conn_01x01_Male, Q1 Conn_01x01_Male

Commit message: complete circuit-2
Parts:
- removed the Clock at (88.4, 127.5)
- removed the GND at (55.9, 140.2)
- removed the Vcc at (55.9, 127.5)
- added Clock: Conn_01x01_Male, Connector_PinHeader_2.54mm:PinHeader_1x01_P2.54mm_Vertical, F.Cu at (90.9, 150.6)
- added GND: Conn_01x01_Male, Connector_PinHeader_2.54mm:PinHeader_1x01_P2.54mm_Vertical, F.Cu at (43.4, 153.9)
- added Vcc: Conn_01x01_Male, Connector_PinHeader_2.54mm:PinHeader_1x01_P2.54mm_Vertical, F.Cu at (43.4, 151.4)
- 74LS00, 74LS73: footprint Connector_PinSocket_2.54mm:PinSocket_2x07_P2.54mm_Vertical -> myFootprint:DIP-14-SMD
- moved 74LS73 32.3 mm to (77.7, 158.2), turned to 0 degrees
- moved Q1 29.6 mm to (90.9, 165.1)
- moved G*** 27.2 mm to (48.8, 161.2)
- moved 74LS00 22.0 mm to (56.6, 158.2), turned to 0 degrees
- moved Q0 18.6 mm to (90.9, 159.1)
- renumbered Q1 to Q0, Q0 to Q1
Connections:
- 74LS73 pad 1: Net-(J3-Pad1) -> CK
- 74LS73 pad 12: Net-(J4-Pad1) -> Net-(J3-Pad1)
- 74LS73 pad 5: CK -> Net-(J3-Pad1)
- 74LS73 pad 9: Net-(J3-Pad1) -> Net-(J4-Pad1)
Routing:
- net GND: track 60.0 -> 9.08 mm, vias 3 -> 4
- net Net-(U1-Pad2): track 21.7 -> 49.2 mm, vias 0 -> 2
- net Net-(J4-Pad1): track 39.6 -> 55.0 mm, vias 0 -> 3
- net Net-(J3-Pad1): track 56.9 -> 61.5 mm, vias 1 -> 5
- net CK: track 17.0 -> 20.2 mm, vias 0 -> 1
- net VCC: track 60.9 -> 60.2 mm
Other:
- board text added: "2020/09/18"
- board text removed: "2020/09/14"

Commit message: add gerber
Parts:
- moved Clock 102.3 mm to (97.5, 48.5)
- moved G*** 102.3 mm to (55.4, 59.1)
- moved GND 102.3 mm to (50.0, 51.8)
- moved Q0 102.3 mm to (97.5, 57.0)
- moved Q1 102.3 mm to (97.5, 63.0)
- moved 74LS00 102.3 mm to (63.2, 56.1)
- moved 74LS73 102.3 mm to (84.3, 56.1)
- moved Vcc 102.3 mm to (50.0, 49.3)
Routing:
- net Net-(J4-Pad1): track 55.0 -> 54.8 mm, vias 3 -> 2
- net Net-(J3-Pad1): vias 5 -> 4
- net GND: vias 4 -> 2
